Commit message: fix: bind xacro prefix argument in TB3 description

File: amr_bringup/urdf/turtlebot3_burger.urdf.xacro (robot description, xacro)
@@ -2,4 +2,5 @@
 <robot xmlns:xacro="http://www.ros.org/wiki/xacro" name="turtlebot3_burger">
   <xacro:arg name="prefix" default=""/>
+  <xacro:property name="prefix" value="$(arg prefix)"/>
   <xacro:property name="base_length" value="0.138"/>
   <xacro:property name="base_width" value="0.178"/>
